Commit message: gimbal control

File: src/controlko_description/urdf/rrbot/rrbot_macro.ros2_control.xacro (robot description, xacro)
@@ -90,23 +90,24 @@
             <param name="motor_type">M3508</param>
       </joint>
-      <!--
-      <joint name="friction_wheel2_joint">
-        <command_interface name="position"/>
-        <state_interface name="position">
-          <param name="initial_value">0.0</param>
-        </state_interface>
-      </joint>
-      -->
-    <!--
-      <joint name="${prefix}friction_wheel1_joint">
+       <joint name="pitch_joint">
             <param name="can_bus">can0</param>
             <param name="tx_id">1</param>
-            <param name="offset">0</param>
-            <param name="motor_type">M3508</param>
-            <command_interface name="velocity"></command_interface>
+            <param name="offset">4649</param>
+            <param name="motor_type">GM6020</param>
+            <command_interface name="position"></command_interface>
             <state_interface name="position"/>
             <state_interface name="velocity"/>
-      </joint>
-    -->
+            <state_interface name="effort"/>
+        </joint>
+        <joint name="yaw_joint">
+            <param name="can_bus">can0</param>
+            <param name="tx_id">2</param>
+            <param name="offset">6668</param>
+            <param name="motor_type">GM6020</param>
+            <command_interface name="position"></command_interface>
+            <state_interface name="position"/>
+            <state_interface name="velocity"/>
+            <state_interface name="effort"/>
+        </joint>
     </ros2_control>
   </xacro:macro>
