Commit message: auto aiming

File: src/my_hardware_interface/urdf/rrbot/rrbot_macro.xacro (robot description, xacro)
@@ -3,85 +3,109 @@
   <xacro:include filename="$(find my_hardware_interface)/urdf/common.xacro" />
   <xacro:macro name="rrbot" params="prefix parent *origin">
-    <!-- LINKS -->
-    <!-- base link -->
+    <!-- 英雄機器人Links -->
     <link name="${prefix}base_link">
-      <!-- Default inertial for Gazebo - copy and edit block from 'common.xacro'
-           to get more realistic behaviour-->
-      <xacro:default_inertial/>
+      <inertial>
+        <origin xyz="0.000276138738735866 0.00564807973459863 0.0606576860440764" rpy="0 0 0" />
+        <mass value="8.78184637370999" />
+        <inertia ixx="0.0148401995915169" ixy="0.000108738329559126" ixz="9.56360986869471E-05" iyy="0.0486787597290484" iyz="-5.79850122096404E-06" izz="0.0557970041196964" />
+      </inertial>
       <visual>
-        <origin xyz="0 0 0.15" rpy="0 0 0" />
+        <origin xyz="0 0 0" rpy="0 0 0" />
         <geometry>
-          <box size="0.3 0.3 0.3"/>
+          <mesh filename="file:///$(find my_hardware_interface)/meshes/hero/base_link.STL" />
         </geometry>
-        <material name="StoglRobotics/Violet"/>
+        <material name="">
+          <color rgba="1 1 1 1" />
+        </material>
       </visual>
       <collision>
-        <origin xyz="0 0 0.15" rpy="0 0 0" />
+        <origin xyz="0 0 0" rpy="0 0 0" />
         <geometry>
-          <box size="0.3 0.3 0.3"/>
+          <mesh filename="file:///$(find my_hardware_interface)/meshes/hero/base_link.STL" />
         </geometry>
       </collision>
     </link>
-    <gazebo reference="${prefix}base_link">
-      <material>Gazebo/Orange</material>
-    </gazebo>
-    <!-- link 1 -->
-    <link name="${prefix}link1">
-      <!-- Default inertial for Gazebo - copy and edit block from 'common.xacro'
-           to get more realistic behaviour-->
-      <xacro:default_inertial/>
+    <link name="${prefix}yaw_link">
+      <inertial>
+        <origin xyz="-0.021742157944887 0.00267307516394979 0.073861518799458" rpy="0 0 0" />
+        <mass value="0.28719249337078" />
+        <inertia ixx="0.000506616303281996" ixy="8.5370250851231E-06" ixz="7.95180991696996E-05" iyy="0.00059114947186763" iyz="-7.95528226323097E-06" izz="9.79994345641336E-05" />
+      </inertial>
       <visual>
-        <origin xyz="0 0 0.25" rpy="0 0 0" />
+        <origin xyz="0 0 0" rpy="0 0 0" />
         <geometry>
-          <cylinder length="0.5" radius="${0.2/2}" />
+          <mesh filename="file:///$(find my_hardware_interface)/meshes/hero/yaw_link.STL" />
         </geometry>
         <material name="StoglRobotics/DarkGrey"/>
       </visual>
       <collision>
-        <origin xyz="0 0 0.25" rpy="0 0 0" />
+        <origin xyz="0 0 0" rpy="0 0 0" />
         <geometry>
-          <cylinder length="0.5" radius="${0.2/2}" />
+          <mesh filename="file:///$(find my_hardware_interface)/meshes/hero/yaw_link.STL" />
         </geometry>
       </collision>
     </link>
-    <gazebo reference="${prefix}link1">
-        <material>Gazebo/Black</material>
-    </gazebo>
-    <!-- link 2 -->
-    <link name="${prefix}link2">
-      <!-- Default inertial for Gazebo - copy and edit block from 'common.xacro'
-           to get more realistic behaviour-->
-      <xacro:default_inertial/>
+    <link name="${prefix}pitch_link">
+      <inertial>
+        <origin xyz="-0.00916934145870887 -0.00928618985529435 0.0240584344921287" rpy="0 0 0" />
+        <mass value="2.16161612754808" />
+        <inertia ixx="0.00188819608033588" ixy="1.90170138375831E-05" ixz="7.20532483480358E-05" iyy="0.00273782224519966" iyz="1.66613979109365E-06" izz="0.00321725364702273" />
+      </inertial>
       <visual>
-        <origin xyz="0 0 0.3" rpy="0 0 0" />
+        <origin xyz="0 0 0" rpy="0 0 0" />
         <geometry>
-          <box size="0.1 0.1 0.6"/>
+          <mesh filename="file:///$(find my_hardware_interface)/meshes/hero/pitch_link.STL" />
         </geometry>
         <material name="StoglRobotics/LightGrey"/>
       </visual>
       <collision>
-        <origin xyz="0 0 0.3" rpy="0 0 0" />
+        <origin xyz="0 0 0" rpy="0 0 0" />
         <geometry>
-          <box size="0.1 0.1 0.6"/>
+          <mesh filename="file:///$(find my_hardware_interface)/meshes/hero/pitch_link.STL" />
         </geometry>
       </collision>
     </link>
-    <gazebo reference="${prefix}link2">
-      <material>Gazebo/Gray</material>
-    </gazebo>
-    <!-- All-zero tool frame. This frame should correspond to the TOOL frame of the robot's controller.) -->
-    <link name="${prefix}tool0" />
-    <!-- tool link -->
-<!-- START Delete if not needed -->
-    <!-- Standard frames for industrial robots. Also useful for manipulators.
-         (ROS-I specs - https://wiki.ros.org/Industrial/Tutorials/WorkingWithRosIndustrialRobotSupportPackages#Standardised_links_.2F_frames)-->
-    <!-- This frame should correspond to the BASE coordinate system of robot's controller.) -->
-    <link name="${prefix}base" />
-    <!-- Frame for mounting EEF models to a manipulator. x+ axis points forward (REP 103). -->
-    <link name="${prefix}flange" />
-<!-- END Delete if not needed  -->
-    <!-- END LINKS -->
-    <!-- JOINTS -->
-    <!-- base_joint fixes base_link to the environment -->
+    <!-- 相機Link -->
+    <link name="${prefix}cam0_link"/>
+    <!-- 摩擦輪Links -->
+    <link name="${prefix}friction_wheel_lf_link">
+      <xacro:default_inertial/>
+      <visual>
+        <origin xyz="0 0 0" rpy="0 0 0" />
+        <geometry>
+          <mesh filename="file:///$(find my_hardware_interface)/meshes/hero/friction_wheel_lf_link.STL" />
+        </geometry>
+        <material name="StoglRobotics/DarkGrey"/>
+      </visual>
+    </link>
+    <!-- 其他摩擦輪 -->
+    <link name="${prefix}friction_wheel_lb_link">
+      <xacro:default_inertial/>
+      <visual>
+        <geometry>
+          <mesh filename="file:///$(find my_hardware_interface)/meshes/hero/friction_wheel_lb_link.STL" />
+        </geometry>
+        <material name="StoglRobotics/DarkGrey"/>
+      </visual>
+    </link>
+    <link name="${prefix}friction_wheel_rf_link">
+      <xacro:default_inertial/>
+      <visual>
+        <geometry>
+          <mesh filename="file:///$(find my_hardware_interface)/meshes/hero/friction_wheel_rf_link.STL" />
+        </geometry>
+        <material name="StoglRobotics/DarkGrey"/>
+      </visual>
+    </link>
+    <link name="${prefix}friction_wheel_rb_link">
+      <xacro:default_inertial/>
+      <visual>
+        <geometry>
+          <mesh filename="file:///$(find my_hardware_interface)/meshes/hero/friction_wheel_rb_link.STL" />
+        </geometry>
+        <material name="StoglRobotics/DarkGrey"/>
+      </visual>
+    </link>
+    <!-- Joints -->
     <joint name="${prefix}base_joint" type="fixed">
       <xacro:insert_block name="origin" />
@@ -89,41 +113,56 @@
       <child link="${prefix}base_link" />
     </joint>
-    <!-- joint 1 -->
-    <joint name="${prefix}joint1" type="revolute">
-      <origin xyz="0 0 0.3" rpy="0 0 0" />
+    <!-- Yaw關節 - 對應ros2_control中的yaw_joint -->
+    <joint name="${prefix}yaw_joint" type="continuous">
+      <origin xyz="0 0 0.216499999999877" rpy="0 0 0" />
       <parent link="${prefix}base_link" />
-      <child link="${prefix}link1" />
+      <child link="${prefix}yaw_link" />
       <axis xyz="0 0 1" />
-      <limit effort="1000" lower="${radians(-380)}" upper="${radians(380)}" velocity="${radians(180)}" />
     </joint>
-    <!-- joint 2 -->
-    <joint name="${prefix}joint2" type="revolute">
-      <origin xyz="0 0 0.5" rpy="0 -${pi/2} 0" />
-      <parent link="${prefix}link1" />
-      <child link="${prefix}link2" />
-      <axis xyz="0 1 0" />
-      <limit effort="1000" lower="${radians(-60)}" upper="${radians(240)}" velocity="${radians(180)}" />
+    <!-- Pitch關節 - 對應ros2_control中的pitch_joint -->
+    <joint name="${prefix}pitch_joint" type="continuous">
+      <origin xyz="0.00383117201995245 0.000563252350000402 0.144999999999997" rpy="0 0 0" />
+      <parent link="${prefix}yaw_link" />
+      <child link="${prefix}pitch_link" />
+      <axis xyz="0 -1 0" />
     </joint>
-    <!-- tool frame - fixed frame -->
-    <joint name="${prefix}link2-tool0" type="fixed">
-      <parent link="${prefix}link2" />
-      <child link="${prefix}tool0" />
-      <origin xyz="0 0 0.6" rpy="0 ${-pi} ${-pi/2}" />
+    <!-- 相機關節 -->
+<joint name="${prefix}cam0_joint" type="fixed">
+  <origin xyz="0.0898857089666096 -0.000941658027797158 0.107797961620051" rpy="0 0 0" />
+  <parent link="${prefix}pitch_link" />
+  <child link="${prefix}cam0_link" />
+</joint>
+<!--光學frame -->
+<link name="${prefix}camera_optical_frame"/>
+<joint name="${prefix}camera_optical_joint" type="fixed">
+  <origin xyz="0 0 0" rpy="${-pi/2} 0 ${-pi/2}" />
+  <parent link="${prefix}cam0_link" />
+  <child link="${prefix}camera_optical_frame" />
+</joint>
+    <!-- 摩擦輪關節 - 對應ros2_control中的friction_wheel1-4 -->
+    <joint name="${prefix}friction_wheel1_joint" type="continuous">
+      <origin xyz="0.103433768203839 0.048100339443673 0.011805507063491" rpy="0 0 0" />
+      <parent link="${prefix}pitch_link" />
+      <child link="${prefix}friction_wheel_lf_link" />
+      <axis xyz="0 0 -1" />
     </joint>
-    <!-- END JOINTS -->
-<!-- START Delete if not needed -->
-    <!-- Standard frames for industrial robots. Also useful for manipulators.
-         (ROS-I specs - https://wiki.ros.org/Industrial/Tutorials/WorkingWithRosIndustrialRobotSupportPackages#Standardised_links_.2F_frames)-->
-    <joint name="${prefix}base_link-base_joint" type="fixed">
-      <origin xyz="0 0 0" rpy="0 0 0" />
-      <parent link="${prefix}base_link" />
-      <child link="${prefix}base" />
+    <joint name="${prefix}friction_wheel2_joint" type="continuous">
+      <origin xyz="0.0364337682038387 0.0481003394436472 0.0118055070632364" rpy="0 0 0" />
+      <parent link="${prefix}pitch_link" />
+      <child link="${prefix}friction_wheel_lb_link" />
+      <axis xyz="0 0 -1" />
     </joint>
-    <joint name="${prefix}tool0-flange_joint" type="fixed">
-      <origin xyz="0 0 0" rpy="0 0 0" />
-      <parent link="${prefix}tool0" />
-      <child link="${prefix}flange" />
+    <joint name="${prefix}friction_wheel3_joint" type="continuous">
+      <origin xyz="0.103433768203875 -0.0498996605563272 0.0118055070634907" rpy="0 0 0" />
+      <parent link="${prefix}pitch_link" />
+      <child link="${prefix}friction_wheel_rf_link" />
+      <axis xyz="0 0 -1" />
     </joint>
-<!-- END Delete if not needed  -->
+    <joint name="${prefix}friction_wheel4_joint" type="continuous">
+      <origin xyz="0.0364337682038749 -0.0498996605563519 0.011805507063236" rpy="0 0 0" />
+      <parent link="${prefix}pitch_link" />
+      <child link="${prefix}friction_wheel_rb_link" />
+      <axis xyz="0 0 -1" />
+    </joint>
   </xacro:macro>
 </robot>

File: src/rm_gimbal_description/urdf/rm_gimbal.urdf.xacro (robot description, xacro)
@@ -2,5 +2,5 @@
 <robot name="rm_gimbal"
   xmlns:xacro="http://ros.org/wiki/xacro">
-  <xacro:arg name="xyz" default="0.10 0 0.05" />
+ <xacro:arg name="xyz" default="0.10 0 0.15" />
   <xacro:arg name="rpy" default="0 0 0" />
   <link name="odom" />
