Commit message: auto aim

File: src/my_hardware_interface/urdf/rrbot/rrbot_macro.ros2_control.xacro (robot description, xacro)
@@ -103,5 +103,5 @@
             <param name="can_bus">can0</param>
             <param name="tx_id">1</param>
-            <param name="offset">6668</param>
+            <param name="offset">0</param>
             <param name="motor_type">GM6020</param>
             <command_interface name="position"></command_interface>

File: src/my_hardware_interface/urdf/rrbot/rrbot_macro.xacro (robot description, xacro)
@@ -6,5 +6,5 @@
     <link name="${prefix}base_link">
       <inertial>
-        <origin xyz="0.000276138738735866 0.00564807973459863 0.0606576860440764" rpy="0 0 0" />
+        <origin xyz="0.0 0.0 0.0" rpy="0 0 0" />
         <mass value="8.78184637370999" />
         <inertia ixx="0.0148401995915169" ixy="0.000108738329559126" ixz="9.56360986869471E-05" iyy="0.0486787597290484" iyz="-5.79850122096404E-06" izz="0.0557970041196964" />
@@ -28,5 +28,5 @@
     <link name="${prefix}yaw_link">
       <inertial>
-        <origin xyz="-0.021742157944887 0.00267307516394979 0.073861518799458" rpy="0 0 0" />
+        <origin xyz="-0.0 0.0 0.0" rpy="0 0 0" />
         <mass value="0.28719249337078" />
         <inertia ixx="0.000506616303281996" ixy="8.5370250851231E-06" ixz="7.95180991696996E-05" iyy="0.00059114947186763" iyz="-7.95528226323097E-06" izz="9.79994345641336E-05" />
@@ -48,5 +48,5 @@
     <link name="${prefix}pitch_link">
       <inertial>
-        <origin xyz="-0.00916934145870887 -0.00928618985529435 0.0240584344921287" rpy="0 0 0" />
+        <origin xyz="0.0 0.0 0.0" rpy="0 0 0" />
         <mass value="2.16161612754808" />
         <inertia ixx="0.00188819608033588" ixy="1.90170138375831E-05" ixz="7.20532483480358E-05" iyy="0.00273782224519966" iyz="1.66613979109365E-06" izz="0.00321725364702273" />
@@ -115,12 +115,12 @@
     <!-- Yaw關節 - 對應ros2_control中的yaw_joint -->
     <joint name="${prefix}yaw_joint" type="continuous">
-      <origin xyz="0 0 0.216499999999877" rpy="0 0 0" />
+      <origin xyz="0 0 0.0" rpy="0 0 0" />
       <parent link="${prefix}base_link" />
       <child link="${prefix}yaw_link" />
-      <axis xyz="0 0 1" />
+      <axis xyz="0 0 -1" />
     </joint>
     <!-- Pitch關節 - 對應ros2_control中的pitch_joint -->
     <joint name="${prefix}pitch_joint" type="continuous">
-      <origin xyz="0.00383117201995245 0.000563252350000402 0.144999999999997" rpy="0 0 0" />
+      <origin xyz="0.0 0.0 0.0" rpy="0 0 0" />
       <parent link="${prefix}yaw_link" />
       <child link="${prefix}pitch_link" />
@@ -129,9 +129,10 @@
     <!-- 相機關節 -->
 <joint name="${prefix}cam0_joint" type="fixed">
-  <origin xyz="0.0898857089666096 -0.000941658027797158 0.107797961620051" rpy="0 0 0" />
+  <origin xyz="0.0 0.0 0.0" rpy="0 0 0" />
   <parent link="${prefix}pitch_link" />
   <child link="${prefix}cam0_link" />
 </joint>
 <!--光學frame -->
+<!--
 <link name="${prefix}camera_optical_frame"/>
 <joint name="${prefix}camera_optical_joint" type="fixed">
@@ -140,4 +141,5 @@
   <child link="${prefix}camera_optical_frame" />
 </joint>
+-->
     <!-- 摩擦輪關節 - 對應ros2_control中的friction_wheel1-4 -->
     <joint name="${prefix}friction_wheel1_joint" type="continuous">

Commit message: Update hardware interface and controller configurations

File: src/my_hardware_interface/urdf/rrbot/rrbot_macro.ros2_control.xacro (robot description, xacro)
@@ -93,5 +93,5 @@
             <param name="can_bus">can0</param>
             <param name="tx_id">2</param>
-            <param name="offset">6108.5</param>
+            <param name="offset">5500</param>
             <param name="motor_type">GM6020</param>
             <command_interface name="position"></command_interface>

File: src/my_hardware_interface/urdf/rrbot/rrbot_macro.xacro (robot description, xacro)
@@ -125,5 +125,5 @@
       <parent link="${prefix}yaw_link" />
       <child link="${prefix}pitch_link" />
-      <axis xyz="0 -1 0" />
+      <axis xyz="0 1 0" />
     </joint>
     <!-- 相機關節 -->

File: src/rm_gimbal_description/urdf/rm_gimbal.urdf.xacro (robot description, xacro)
@@ -2,5 +2,5 @@
 <robot name="rm_gimbal"
   xmlns:xacro="http://ros.org/wiki/xacro">
- <xacro:arg name="xyz" default="0.10 0 0.15" />
+ <xacro:arg name="xyz" default="0.10 -1 0.15" />
   <xacro:arg name="rpy" default="0 0 0" />
   <link name="odom" />
